File: main.brd (EAGLE design)
At the start: 100 x 58 mm, 94 parts, among them J1 FH34SRJ-24S-0.5SH, J2 ICSP, J3 USB, Q1 NMOS, Q10 PMOS, Q2 NMOS, Q3 PMOS, Q4 PMOS, Q5 NMOSL, Q6 NMOSL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

Commit message: Production version
Parts:
- H1, H2, H3, H4: value (none) -> MOUNT
- moved C2 6.32 mm to (71.0, 12.1), turned to 0 degrees
- moved R1 2.03 mm to (61.1, 2.92)
- moved R2 2.03 mm to (61.1, 5.97)
- moved C3 2.03 mm to (63.1, 4.45)
- moved J3 0.25 mm to (36.8, 2.79)
- moved R6 0.25 mm to (7.37, 1.65)
- moved R7 0.25 mm to (7.37, 3.68)
- moved C18 0.25 mm to (37.1, 5.21)
- moved F2 0.25 mm to (40.6, 5.21)
Routing:
- net USB_VBUS: track 3.58 -> 118.2 mm, vias 0 -> 5
- net 3.3V: track 46.8 -> 158.6 mm, vias 0 -> 3
- net GREEN_LED_EN: track 0.00 -> 76.8 mm, vias 0 -> 2
- net RED_LED_EN: track 0.00 -> 73.7 mm, vias 0 -> 2
- net MCU_POWERSW: track 0.00 -> 66.9 mm, vias 0 -> 1
- net CHG_LED_R: track 0.00 -> 66.4 mm, vias 0 -> 2
- net CHG_LED_G: track 0.00 -> 63.3 mm, vias 0 -> 2
- net MCU_MEASURESW: track 0.00 -> 58.7 mm, vias 0 -> 1
- net VIN: track 17.7 -> 52.6 mm, vias 0 -> 1
- net SCD_PDN: track 0.00 -> 33.7 mm
- net VBAT: track 30.3 -> 62.7 mm
- net !MCLR: track 0.00 -> 31.2 mm, vias 0 -> 2
- net SCD_RDY: track 0.00 -> 29.1 mm
- net EPD_!RST: track 15.0 -> 37.7 mm
- net VBAT_MEASURE_EN: track 0.00 -> 22.2 mm, vias 0 -> 2
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- added copper zone on layer 1, net GND
- added copper zone on layer 16, net GND
- added copper zone on layer 16, net LOGO
Other:
- board text added: "+"
- board text added: "1"
- board text added: "CO2 Station ©2021 BlockWorker blockworker.de"
- board text added: "JLCJLCJLCJLC"
