File: main.sch (EAGLE design)
At the start: 94 parts, among them J1 FH34SRJ-24S-0.5SH, J2 ICSP, J3 USB, Q1 NMOS, Q10 PMOS, Q2 NMOS, Q3 PMOS, Q4 PMOS, Q5 NMOSL, Q6 NMOSL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

Commit message: Production version
Parts:
- H1, H2, H3, H4: value (none) -> MOUNT
Changed lines of the file:
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@@
 <attribute name="TP_SIGNAL_NAME" value="EPD_PDN"/>
 </part>
-<part name="H1" library="BW-Connectors" deviceset="7466313R" device=""/>
-<part name="H2" library="BW-Connectors" deviceset="7466313R" device=""/>
-<part name="H3" library="BW-Connectors" deviceset="7466313R" device=""/>
-<part name="H4" library="BW-Connectors" deviceset="7466313R" device=""/>
+<part name="H1" library="BW-Connectors" deviceset="7466313R" device="" value="MOUNT"/>
+<part name="H2" library="BW-Connectors" deviceset="7466313R" device="" value="MOUNT"/>
+<part name="H3" library="BW-Connectors" deviceset="7466313R" device="" value="MOUNT"/>
+<part name="H4" library="BW-Connectors" deviceset="7466313R" device="" value="MOUNT"/>
 </parts>
 <sheets>
@@
 <net name="USB_VBUS" class="0">
 <segment>
-<pinref part="C18" gate="G$1" pin="1"/>
-<wire x1="-88.9" y1="-109.22" x2="-88.9" y2="-106.68" width="0.1524" layer="91"/>
 <pinref part="U2" gate="G$1" pin="VCC"/>
+<wire x1="-96.52" y1="-106.68" x2="-88.9" y2="-106.68" width="0.1524" layer="91"/>
 <wire x1="-88.9" y1="-106.68" x2="-66.04" y2="-106.68" width="0.1524" layer="91"/>
 <wire x1="-66.04" y1="-106.68" x2="-66.04" y2="-137.16" width="0.1524" layer="91"/>
@@
 <wire x1="-50.8" y1="-137.16" x2="-50.8" y2="-154.94" width="0.1524" layer="91"/>
 <pinref part="F2" gate="G$1" pin="2"/>
-<wire x1="-96.52" y1="-106.68" x2="-88.9" y2="-106.68" width="0.1524" layer="91"/>
-<junction x="-88.9" y="-106.68"/>
 <pinref part="TP6" gate="G$1" pin="TP"/>
 <wire x1="-66.04" y1="-104.14" x2="-66.04" y2="-106.68" width="0.1524" layer="91"/>
 <junction x="-66.04" y="-106.68"/>
-</segment>
-<segment>
+<pinref part="C18" gate="G$1" pin="1"/>
+<wire x1="-88.9" y1="-109.22" x2="-88.9" y2="-106.68" width="0.1524" layer="91"/>
+<junction x="-88.9" y="-106.68"/>
+<wire x1="-66.04" y1="-106.68" x2="-63.5" y2="-106.68" width="0.1524" layer="91"/>
+<label x="-63.5" y="-106.68" size="1.778" layer="95"/>
+</segment>
+<segment>
